File: microswitch-dpad.kicad_pcb (KiCad board)
At the start: 2 copper layers, 18.9 x 27.7 mm, 12 parts, among them J1 Conn_01x05_Socket, J2 Conn_01x03_Socket, U1 D2LS-21_C3823622, U2 D2LS-21_C3823622, U3 D2LS-21_C3823622, U4 D2LS-21_C3823622

Commit message: added in do, fixed some traces
Parts:
- removed LOGO1: **REF, ct-kicad:awesome-logo
- added LOGO2: **REF, ct-kicad:awesome-logo, B.Cu at (131.4, 92.2)
- J2: footprint Connector_PinSocket_2.54mm:PinSocket_1x03_P2.54mm_Vertical -> Connector_PinSocket_2.54mm:PinSocket_1x04_P2.54mm_Vertical
Connections:
- D4 pad 3: unconnected-(D4-DOUT-Pad3) -> DO
Routing:
- net DO: track 0.00 -> 28.9 mm, vias 0 -> 2
- net row: track 35.7 -> 28.3 mm, vias 4 -> 3
- net Net-(D2-DOUT): track 13.4 -> 11.4 mm
- net col4: track 26.3 -> 25.4 mm
- net col1: track 11.8 -> 12.7 mm
- net col2: track 11.9 -> 12.5 mm
- net +5V: track 48.1 -> 47.9 mm, vias 6 -> 5
- net GND: vias 0 -> 10
- added copper zone on B.Cu, net GND
Other:
- board size 18.9 x 27.7 mm -> 18.9 x 27.8 mm
- board text added: "C4 C3 C2 C1 RW"
- board text added: "DO DI 5V GD"
- board text added: "DPAD"
- board text added: "INATOR"
- board text added: "v1.0"
