File: microswitch-dpad.kicad_pcb (KiCad board)
At the start: 2 copper layers, 18.9 x 27.8 mm, 12 parts, among them J1 Conn_01x05_Socket, J2 Conn_01x03_Socket, U1 D2LS-21_C3823622, U2 D2LS-21_C3823622, U3 D2LS-21_C3823622, U4 D2LS-21_C3823622

Commit message: production submitted
Parts:
- removed J2: Conn_01x03_Socket, Connector_PinSocket_2.54mm:PinSocket_1x04_P2.54mm_Vertical
- J1: value Conn_01x05_Socket -> Conn_01x09_Socket; footprint Connector_PinSocket_2.54mm:PinSocket_1x05_P2.54mm_Vertical -> Connector_PinSocket_1.27mm:PinSocket_1x09_P1.27mm_Vertical
- moved J1 0.75 mm to (132.1, 81.5)
- moved C1 0.49 mm to (133.9, 83.3)
Connections:
- J1 pad 1: row -> GND
- J1 pad 2: col1 -> +5V
- J1 pad 3: col2 -> DI
- J1 pad 4: col3 -> DO
- J1 pad 5: col4 -> row
Routing:
- net GND: track 0.00 -> 10.5 mm, vias 10 -> 9
- net DI: track 22.5 -> 16.0 mm
- net DO: track 28.9 -> 23.6 mm, vias 2 -> 1
- net +5V: track 47.9 -> 43.1 mm
- net col1: track 12.7 -> 8.88 mm
- net col2: track 12.5 -> 10.3 mm
- net row: track 28.3 -> 29.6 mm, vias 3 -> 4
- net col4: track 25.4 -> 24.6 mm
- net col3: track 20.5 -> 19.7 mm
- net Net-(D3-DOUT): track 17.2 -> 16.5 mm
Other:
- board size 18.9 x 27.8 mm -> 18.9 x 22.4 mm
- board text added: "4 3 2 1 R O I 5 G"
- board text removed: "C4 C3 C2 C1 RW"
- board text removed: "DO DI 5V GD"
