File: microswitch-dpad.kicad_sch (KiCad schematic)
At the start: 12 parts, among them J1 Conn_01x05_Socket, J2 Conn_01x03_Socket, U1 D2LS-21_C3823622, U2 D2LS-21_C3823622, U3 D2LS-21_C3823622, U4 D2LS-21_C3823622

Commit message: added in do, fixed some traces
Parts:
- removed LOGO1: **REF, ct-kicad:awesome-logo, symbol ct-kicad:awesome-logo
- added LOGO2: **REF, ct-kicad:awesome-logo, symbol ct-kicad:awesome-logo
- J2: footprint Connector_PinSocket_2.54mm:PinSocket_1x03_P2.54mm_Vertical -> Connector_PinSocket_2.54mm:PinSocket_1x04_P2.54mm_Vertical; symbol Connector:Conn_01x03_Socket -> Connector:Conn_01x04_Socket; now in the parts list
Connections:
- net DO: now reaches D4.3 (DOUT)
- net DO: now also J2.4 (Pin_4)
- no-connect marks 1 -> 0
Changed lines of the file:
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@@
 		(color 0 0 0 0)
 	)
-	(no_connect
-		(at 184.15 57.15)
-	)
 	(wire
 		(pts
@@
 	(wire
 		(pts
+			(xy 88.9 66.04) (xy 91.44 66.04)
+		)
+		(stroke
+			(width 0)
+			(type default)
+		)
+	)
+	(wire
+		(pts
 			(xy 101.6 99.06) (xy 105.41 99.06)
 		)
@@
 		(pts
 			(xy 143.51 49.53) (xy 154.94 49.53)
+		)
+		(stroke
+			(width 0)
+			(type default)
+		)
+	)
+	(wire
+		(pts
+			(xy 184.15 57.15) (xy 189.23 57.15)
 		)
 		(stroke
@@
 		)
 	)
+	(global_label "DO"
+		(shape input)
+		(at 91.44 66.04 0)
+		(fields_autoplaced yes)
+		(effects
+			(font
+				(size 1.27 1.27)
+			)
+			(justify left)
+		)
+		(property "Intersheetrefs" "${INTERSHEET_REFS}"
+			(at 97.0257 66.04 0)
+			(effects
+				(font
+					(size 1.27 1.27)
+				)
+				(justify left)
+				(hide yes)
+			)
+		)
+	)
 	(global_label "col4"
 		(shape input)
@@
 		(property "Intersheetrefs" "${INTERSHEET_REFS}"
 			(at 112.5075 88.9 0)
+			(effects
+				(font
+					(size 1.27 1.27)
+				)
+				(justify left)
+				(hide yes)
+			)
+		)
+	)
+	(global_label "DO"
+		(shape output)
+		(at 189.23 57.15 0)
+		(fields_autoplaced yes)
+		(effects
+			(font
+				(size 1.27 1.27)
+			)
+			(justify left)
+		)
+		(property "Intersheetrefs" "${INTERSHEET_REFS}"
+			(at 194.8157 57.15 0)
 			(effects
 				(font
@@
 	)
 	(symbol
+		(lib_id "ct-kicad:awesome-logo")
+		(at 181.61 38.1 0)
+		(unit 1)
+		(exclude_from_sim no)
+		(in_bom no)
+		(on_board yes)
+		(dnp no)
+		(fields_autoplaced yes)
+		(property "Reference" "LOGO2"
+			(at 184.15 36.8299 0)
+			(effects
+				(font
+					(size 1.27 1.27)
+				)
+				(justify left)
+			)
+		)
+		(property "Value" "**REF"
+			(at 184.15 39.3699 0)
+			(effects
+				(font
+					(size 1.27 1.27)
+				)
+				(justify left)
+			)
+		)
+		(property "Footprint" "ct-kicad:awesome-logo"
+			(at 181.61 38.1 0)
+			(effects
+				(font
+					(size 1.27 1.27)
+				)
+				(hide yes)
+			)
+		)
+		(property "Datasheet" ""
+			(at 181.61 38.1 0)
+			(effects
+				(font
+					(size 1.27 1.27)
+				)
+				(hide yes)
+			)
+		)
+		(property "Description" "the crazymittens logo"
+			(at 181.61 38.1 0)
+			(effects
+				(font
+					(size 1.27 1.27)
+				)
+				(hide yes)
+			)
+		)
+		(instances
+			(project "microswitch-dpad"
+				(path "/4167ffbf-dac9-455c-9662-acf6ff0b6a94"
+					(reference "LOGO2")
+					(unit 1)
+				)
+			)
+		)
+	)
+	(symbol
 		(lib_id "power:GND")
 		(at 91.44 73.66 90)
@@
 	)
 	(symbol
-		(lib_id "Connector:Conn_01x03_Socket")
+		(lib_id "Connector:Conn_01x04_Socket")
 		(at 83.82 71.12 180)
 		(unit 1)
 		(exclude_from_sim no)
-		(in_bom no)
+		(in_bom yes)
 		(on_board yes)
 		(dnp no)
 		(fields_autoplaced yes)
 		(property "Reference" "J2"
+			(at 84.455 60.96 0)
+			(effects
+				(font
+					(size 1.27 1.27)
+				)
+			)
+		)
+		(property "Value" "Conn_01x03_Socket"
 			(at 84.455 63.5 0)
 			(effects
@@
 			)
 		)
-		(property "Value" "Conn_01x03_Socket"
-			(at 84.455 66.04 0)
-			(effects
-				(font
-					(size 1.27 1.27)
-				)
-			)
-		)
-		(property "Footprint" "Connector_PinSocket_2.54mm:PinSocket_1x03_P2.54mm_Vertical"
+		(property "Footprint" "Connector_PinSocket_2.54mm:PinSocket_1x04_P2.54mm_Vertical"
 			(at 83.82 71.12 0)
 			(effects
@@
 			)
 		)
-		(property "Description" "Generic connector, single row, 01x03, script generated"
+		(property "Description" "Generic connector, single row, 01x04, script generated"
 			(at 83.82 71.12 0)
 			(effects
@@
 		)
 		(pin "2"
+		)
+		(pin "4"
 		)
 		(instances
@@
 					(unit 1)
 				)
-			)
-		)
-	)
-	(symbol
-		(lib_id "ct-kicad:awesome-logo")
-		(at 167.64 38.1 0)
-		(unit 1)
-		(exclude_from_sim no)
-		(in_bom no)
-		(on_board yes)
-		(dnp no)
-		(fields_autoplaced yes)
-		(property "Reference" "LOGO1"
-			(at 170.18 36.8299 0)
-			(effects
-				(font
-					(size 1.27 1.27)
-				)
-				(justify left)
-			)
-		)
-		(property "Value" "**REF"
-			(at 170.18 39.3699 0)
-			(effects
-				(font
-					(size 1.27 1.27)
-				)
-				(justify left)
-			)
-		)
-		(property "Footprint" "ct-kicad:awesome-logo"
-			(at 167.64 38.1 0)
-			(effects
-				(font
-					(size 1.27 1.27)
-				)
-				(hide yes)
-			)
-		)
-		(property "Datasheet" ""
-			(at 167.64 38.1 0)
-			(effects
-				(font
-					(size 1.27 1.27)
-				)
-				(hide yes)
-			)
-		)
-		(property "Description" "the crazymittens logo"
-			(at 167.64 38.1 0)
-			(effects
-				(font
-					(size 1.27 1.27)
-				)
-				(hide yes)
-			)
-		)
-		(instances
-			(project "microswitch-dpad"
-				(path "/4167ffbf-dac9-455c-9662-acf6ff0b6a94"
-					(reference "LOGO1")
-					(unit 1)
-				)

Commit message: production submitted
Parts:
- removed J1: Conn_01x05_Socket, Connector_PinSocket_2.54mm:PinSocket_1x05_P2.54mm_Vertical, symbol Connector:Conn_01x05_Socket
- removed J2: Conn_01x03_Socket, Connector_PinSocket_2.54mm:PinSocket_1x04_P2.54mm_Vertical, symbol Connector:Conn_01x04_Socket
- added J1: Conn_01x09_Socket, Connector_PinSocket_1.27mm:PinSocket_1x09_P1.27mm_Vertical, symbol Connector:Conn_01x09_Socket
Connections:
- net +5V: now also J1.2 (Pin_2)
- net DI: now also J1.3 (Pin_3)
- net DO: now also J1.4 (Pin_4)
- net GND: now also J1.1 (Pin_1)
- net col1: now also J1.6 (Pin_6)
- net col2: now also J1.7 (Pin_7)
- net col3: now also J1.8 (Pin_8)
- net col4: now also J1.9 (Pin_9)
- net row: now also J1.5 (Pin_5)
